Commit message: nuevos_objetos

File: kautham/battery_task_models/battery_new.urdf (robot description, URDF)
Before this commit: robot battery_new, 1 links, 0 joints
Links:
- link base: geometry collision cylinder length=0.059 radius=0.0165; visual cylinder length=0.059 radius=0.0165

File: kautham/battery_task_models/battery_old.urdf (robot description, URDF)
Before this commit: robot battery_old, 1 links, 0 joints
Links:
- link base: geometry collision cylinder length=0.059 radius=0.0165; visual cylinder length=0.059 radius=0.0165

File: kautham/battery_task_models/device_box.urdf (robot description, URDF)
Before this commit: robot device_box, 1 links, 0 joints
Links:
- link base: geometry collision box size=0.006 0.070 0.062; collision box size=0.006 0.070 0.062

File: kautham/battery_task_models/lid.urdf (robot description, URDF)
Before this commit: robot lid, 1 links, 0 joints
Links:
- link base: geometry collision box size=0.040 0.020 0.015; collision box size=0.072 0.072 0.008

File: kautham/battery_task_models/new_battery_box.urdf (robot description, URDF)
Before this commit: robot new_battery_box, 1 links, 0 joints
Links:
- link base: geometry collision box size=0.005 0.070 0.025; collision box size=0.005 0.070 0.025

File: kautham/battery_task_models/used_battery_box.urdf (robot description, URDF)
Before this commit: robot used_battery_box, 1 links, 0 joints
Links:
- link base: geometry collision box size=0.005 0.070 0.025; collision box size=0.005 0.070 0.025
