Commit message: actualizado el dominio

File: kautham/battery_task_models/device_box.urdf (robot description, URDF)
Before this commit: robot device_box, 1 links, 0 joints
Links:
- link base: geometry collision box size=0.070 0.070 0.003; visual box size=0.006 0.070 0.062

File: kautham/battery_task_models/new_battery_box.urdf (robot description, URDF)
Before this commit: robot new_battery_box, 1 links, 0 joints
Links:
- link base: geometry collision box size=0.070 0.070 0.003; visual box size=0.005 0.070 0.025

File: kautham/battery_task_models/used_battery_box.urdf (robot description, URDF)
Before this commit: robot used_battery_box, 1 links, 0 joints
Links:
- link base: geometry collision box size=0.070 0.070 0.003; visual box size=0.005 0.070 0.025
